Commit message: Update Spot gripper

File: bd_spot_gripper/urdf/spot_gripper.urdf (robot description, URDF)
Before this commit: robot spot_gripper, 3 links, 2 joints
Links:
- link arm_link_fngr: geometry collision mesh filename=../meshes/collision/left_finger.obj; collision mesh filename=../meshes/collision/left_hinge.obj
- link arm_link_wr1: geometry collision mesh filename=../meshes/collision/arm_link_wr1.obj; collision mesh filename=../meshes/collision/front_jaw.obj
